Commit message: joint state

File: src/launch/krb2026b_launch/urdf/krb2026b.urdf.xacro (robot description, xacro)
@@ -50,3 +50,18 @@
   <xacro:swerve steer_name="swerve_steer_2" wheel_name="swerve_wheel_2" x="-0.173" y="-0.173"/>
   <xacro:swerve steer_name="swerve_steer_3" wheel_name="swerve_wheel_3" x="0.173"  y="-0.173"/>
+  <!-- ==================== -->
+  <!-- Lidar frames         -->
+  <!-- ==================== -->
+  <link name="lidar_front"/>
+  <joint name="base_link_to_lidar_front" type="fixed">
+    <parent link="base_link"/>
+    <child link="lidar_front"/>
+    <origin xyz="0.2 0 0" rpy="0 0 0"/>
+  </joint>
+  <link name="lidar_rear"/>
+  <joint name="base_link_to_lidar_rear" type="fixed">
+    <parent link="base_link"/>
+    <child link="lidar_rear"/>
+    <origin xyz="-0.2 0 0" rpy="0 0 3.1415926535"/>
+  </joint>
 </robot>

Commit message: fix urdf

File: src/launch/krb2026b_launch/urdf/krb2026b.urdf.xacro (robot description, xacro)
@@ -13,11 +13,11 @@
   <!-- Wheel module macro    -->
   <!-- ==================== -->
-  <xacro:macro name="swerve" params="steer_name wheel_name x y">
+  <xacro:macro name="swerve" params="wheel_base_name wheel_name x y">
     <!-- steer link -->
-    <link name="${steer_name}_link" />
+    <link name="${wheel_base_name}_link" />
     <!-- steer joint -->
-    <joint name="${steer_name}" type="continuous">
+    <joint name="${wheel_base_name}" type="continuous">
       <parent link="base_link"/>
-      <child link="${steer_name}_link"/>
+      <child link="${wheel_base_name}_link"/>
       <origin xyz="${x} ${y} ${wheel_radius}" rpy="0 0 0"/>
       <axis xyz="0 0 1"/>
@@ -37,5 +37,5 @@
     <!-- wheel joint -->
     <joint name="${wheel_name}" type="continuous">
-      <parent link="${steer_name}_link"/>
+      <parent link="${wheel_base_name}_link"/>
       <child link="${wheel_name}_link"/>
       <origin xyz="0 0 0" rpy="0 0 0"/>
@@ -46,8 +46,8 @@
   <!-- Wheel instances       -->
   <!-- ==================== -->
-  <xacro:swerve steer_name="swerve_steer_0" wheel_name="swerve_wheel_0" x="0.173"  y="0.173"/>
-  <xacro:swerve steer_name="swerve_steer_1" wheel_name="swerve_wheel_1" x="-0.173" y="0.173"/>
-  <xacro:swerve steer_name="swerve_steer_2" wheel_name="swerve_wheel_2" x="-0.173" y="-0.173"/>
-  <xacro:swerve steer_name="swerve_steer_3" wheel_name="swerve_wheel_3" x="0.173"  y="-0.173"/>
+  <xacro:swerve wheel_base_name="swerve_wheel_base_0" wheel_name="swerve_wheel_0" x="0.173"  y="0.173"/>
+  <xacro:swerve wheel_base_name="swerve_wheel_base_1" wheel_name="swerve_wheel_1" x="-0.173" y="0.173"/>
+  <xacro:swerve wheel_base_name="swerve_wheel_base_2" wheel_name="swerve_wheel_2" x="-0.173" y="-0.173"/>
+  <xacro:swerve wheel_base_name="swerve_wheel_base_3" wheel_name="swerve_wheel_3" x="0.173"  y="-0.173"/>
   <!-- ==================== -->
   <!-- Lidar frames         -->

Commit message: add stl

File: src/launch/krb2026b_launch/urdf/krb2026b.urdf.xacro (robot description, xacro)
@@ -6,8 +6,19 @@
   <xacro:property name="wheel_radius" value="0.0375"/>
   <xacro:property name="wheel_width"  value="0.02"/>
+  <material name="white">
+    <color rgba="1.000 1.000 1.000 1.0"/>
+  </material>
   <!-- ==================== -->
   <!-- Base link             -->
   <!-- ==================== -->
-  <link name="base_link"/>
+  <link name="base_link">
+    <visual>
+      <origin xyz="0 0 0" rpy="0 0 0"/>
+      <geometry>
+        <mesh filename="package://krb2026b_launch/meshes/base_link.stl"/>
+      </geometry>
+      <material name="white"/>
+    </visual>
+  </link>
   <!-- ==================== -->
   <!-- Wheel module macro    -->
@@ -15,5 +26,13 @@
   <xacro:macro name="swerve" params="wheel_base_name wheel_name x y">
     <!-- steer link -->
-    <link name="${wheel_base_name}_link" />
+    <link name="${wheel_base_name}_link">
+      <visual>
+        <origin xyz="0 0 0.17485" rpy="0 0 0"/>
+        <geometry>
+          <mesh filename="package://krb2026b_launch/meshes/wheel.stl"/>
+        </geometry>
+        <material name="white"/>
+      </visual>
+    </link>
     <!-- steer joint -->
     <joint name="${wheel_base_name}" type="continuous">
@@ -65,3 +84,83 @@
     <origin xyz="-0.2 0 0" rpy="0 0 3.1415926535"/>
   </joint>
+  <joint name="belt_launcher" type="prismatic">
+    <origin xyz="-0.15555731148 0.0 0.18967226953" rpy="0.0 -0.43633231299 0.0"/>
+    <axis xyz="1 0 0"/>
+    <parent link="base_link"/>
+    <child link="belt_launcher_link"/>
+    <limit lower="0.0" upper="0.5" effort="0" velocity="0"/>
+  </joint>
+  <link name="belt_launcher_link">
+    <visual>
+      <origin xyz="0 0 0" rpy="0 0 0"/>
+      <geometry>
+        <mesh filename="package://krb2026b_launch/meshes/belt_launcher.stl"/>
+      </geometry>
+      <material name="white"/>
+    </visual>
+  </link>
+  <joint name="collector_arm_left" type="revolute">
+    <origin xyz="-0.052075 0.233296 0.193222" rpy="0.0 0.0 0.0"/>
+    <axis xyz="0 1 0"/>
+    <parent link="base_link"/>
+    <child link="collector_arm_left_link"/>
+    <limit lower="-3.14159" upper="3.14159" effort="0" velocity="0"/>
+  </joint>
+  <link name="collector_arm_left_link">
+    <visual>
+      <origin xyz="0 0 0" rpy="0 0 0"/>
+      <geometry>
+        <mesh filename="package://krb2026b_launch/meshes/collector_arm_left.stl"/>
+      </geometry>
+      <material name="white"/>
+    </visual>
+  </link>
+  <joint name="collector_hand_left" type="revolute">
+    <origin xyz="-0.149379 0.02 0.028125" rpy="0.0 0.0 0.0"/>
+    <axis xyz="0 0 1"/>
+    <parent link="collector_arm_left_link"/>
+    <child link="collector_hand_left_link"/>
+    <limit lower="-3.14159" upper="3.14159" effort="0" velocity="0"/>
+  </joint>
+  <link name="collector_hand_left_link">
+    <visual>
+      <origin xyz="0 0 0" rpy="0 0 0"/>
+      <geometry>
+        <mesh filename="package://krb2026b_launch/meshes/collector_hand_left.stl"/>
+      </geometry>
+      <material name="white"/>
+    </visual>
+  </link>
+  <joint name="collector_arm_right" type="revolute">
+    <origin xyz="-0.052075 -0.233296 0.193222" rpy="0.0 0.0 0.0"/>
+    <axis xyz="0 1 0"/>
+    <parent link="base_link"/>
+    <child link="collector_arm_right_link"/>
+    <limit lower="-3.14159" upper="3.14159" effort="0" velocity="0"/>
+  </joint>
+  <link name="collector_arm_right_link">
+    <visual>
+      <origin xyz="0 0 0" rpy="0 0 0"/>
+      <geometry>
+        <mesh filename="package://krb2026b_launch/meshes/collector_arm_right.stl"/>
+      </geometry>
+      <material name="white"/>
+    </visual>
+  </link>
+  <joint name="collector_hand_right" type="revolute">
+    <origin xyz="-0.149379 -0.02 0.028125" rpy="0.0 0.0 0.0"/>
+    <axis xyz="0 0 -1"/>
+    <parent link="collector_arm_right_link"/>
+    <child link="collector_hand_right_link"/>
+    <limit lower="-3.14159" upper="3.14159" effort="0" velocity="0"/>
+  </joint>
+  <link name="collector_hand_right_link">
+    <visual>
+      <origin xyz="0 0 0" rpy="0 0 0"/>
+      <geometry>
+        <mesh filename="package://krb2026b_launch/meshes/collector_hand_right.stl"/>
+      </geometry>
+      <material name="white"/>
+    </visual>
+  </link>
 </robot>

Commit message: fix param

File: src/launch/krb2026b_launch/urdf/krb2026b.urdf.xacro (robot description, xacro)
@@ -40,4 +40,13 @@
       <child link="${wheel_base_name}_link"/>
       <origin xyz="${x} ${y} ${wheel_radius}" rpy="0 0 0"/>
+      <axis xyz="0 0 1"/>
+    </joint>
+    <!-- as5600 link -->
+    <link name="${wheel_base_name}_as5600_link"/>
+    <!-- as5600 joint -->
+    <joint name="${wheel_base_name}_as5600" type="continuous">
+      <parent link="base_link"/>
+      <child link="${wheel_base_name}_as5600_link"/>
+      <origin xyz="${x} ${y} 0.1" rpy="0 0 0"/>
       <axis xyz="0 0 1"/>
     </joint>

Commit message: update some

File: src/launch/krb2026b_launch/urdf/krb2026b.urdf.xacro (robot description, xacro)
@@ -48,5 +48,5 @@
       <parent link="base_link"/>
       <child link="${wheel_base_name}_as5600_link"/>
-      <origin xyz="${x} ${y} 0.1" rpy="0 0 0"/>
+      <origin xyz="${x} ${y} 0.16" rpy="0 0 0"/>
       <axis xyz="0 0 1"/>
     </joint>

Commit message: fix visual

File: src/launch/krb2026b_launch/urdf/krb2026b.urdf.xacro (robot description, xacro)
@@ -28,5 +28,5 @@
     <link name="${wheel_base_name}_link">
       <visual>
-        <origin xyz="0 0 0.17485" rpy="0 0 0"/>
+        <origin xyz="0 0 0.14" rpy="0 0 0"/>
         <geometry>
           <mesh filename="package://krb2026b_launch/meshes/wheel.stl"/>

Commit message: latest

File: src/launch/krb2026b_launch/urdf/krb2026b.urdf.xacro (robot description, xacro)
@@ -127,5 +127,5 @@
   <joint name="collector_hand_left" type="revolute">
     <origin xyz="-0.149379 0.02 0.028125" rpy="0.0 0.0 0.0"/>
-    <axis xyz="0 0 1"/>
+    <axis xyz="0 0 -1"/>
     <parent link="collector_arm_left_link"/>
     <child link="collector_hand_left_link"/>
@@ -159,5 +159,5 @@
   <joint name="collector_hand_right" type="revolute">
     <origin xyz="-0.149379 -0.02 0.028125" rpy="0.0 0.0 0.0"/>
-    <axis xyz="0 0 -1"/>
+    <axis xyz="0 0 1"/>
     <parent link="collector_arm_right_link"/>
     <child link="collector_hand_right_link"/>

Commit message: latest

File: src/launch/krb2026b_launch/urdf/krb2026b.urdf.xacro (robot description, xacro)
@@ -81,9 +81,15 @@
   <!-- Lidar frames         -->
   <!-- ==================== -->
-  <link name="lidar_front"/>
-  <joint name="base_link_to_lidar_front" type="fixed">
+  <link name="lidar_right"/>
+  <joint name="base_link_to_lidar_right" type="fixed">
     <parent link="base_link"/>
-    <child link="lidar_front"/>
-    <origin xyz="0.2 0 0" rpy="0 0 0"/>
+    <child link="lidar_right"/>
+    <origin xyz="0.0 -0.184 0" rpy="0 0 1.5708"/>
+  </joint>
+  <link name="lidar_left"/>
+  <joint name="base_link_to_lidar_left" type="fixed">
+    <parent link="base_link"/>
+    <child link="lidar_left"/>
+    <origin xyz="0.0 0.184 0" rpy="0 0 -1.5708"/>
   </joint>
   <link name="lidar_rear"/>
@@ -91,5 +97,5 @@
     <parent link="base_link"/>
     <child link="lidar_rear"/>
-    <origin xyz="-0.2 0 0" rpy="0 0 3.1415926535"/>
+    <origin xyz="-0.3 -0.07 0.1" rpy="0 0 3.1415926535"/>
   </joint>
   <joint name="belt_launcher" type="prismatic">

Commit message: fix belt launcher

File: src/launch/krb2026b_launch/urdf/krb2026b.urdf.xacro (robot description, xacro)
@@ -85,5 +85,5 @@
     <parent link="base_link"/>
     <child link="lidar_right"/>
-    <origin xyz="0.0 -0.184 0" rpy="0 0 1.5708"/>
+    <origin xyz="0.0 -0.184 0" rpy="0 0 -1.5708"/>
   </joint>
   <link name="lidar_left"/>
@@ -91,5 +91,5 @@
     <parent link="base_link"/>
     <child link="lidar_left"/>
-    <origin xyz="0.0 0.184 0" rpy="0 0 -1.5708"/>
+    <origin xyz="0.0 0.184 0" rpy="0 0 1.5708"/>
   </joint>
   <link name="lidar_rear"/>
@@ -99,10 +99,9 @@
     <origin xyz="-0.3 -0.07 0.1" rpy="0 0 3.1415926535"/>
   </joint>
-  <joint name="belt_launcher" type="prismatic">
+  <joint name="belt_launcher" type="continuous">
     <origin xyz="-0.15555731148 0.0 0.18967226953" rpy="0.0 -0.43633231299 0.0"/>
-    <axis xyz="1 0 0"/>
+    <axis xyz="0 1 0"/>
     <parent link="base_link"/>
     <child link="belt_launcher_link"/>
-    <limit lower="0.0" upper="0.5" effort="0" velocity="0"/>
   </joint>
   <link name="belt_launcher_link">

Commit message: 実機調整

File: src/launch/krb2026b_launch/urdf/krb2026b.urdf.xacro (robot description, xacro)
@@ -97,5 +97,5 @@
     <parent link="base_link"/>
     <child link="lidar_rear"/>
-    <origin xyz="-0.3 -0.07 0.1" rpy="0 0 3.1415926535"/>
+    <origin xyz="-0.288 -0.07 0.1" rpy="0 0 3.1415926535"/>
   </joint>
   <joint name="belt_launcher" type="continuous">

Commit message: opi latest

File: src/launch/krb2026b_launch/urdf/krb2026b.urdf.xacro (robot description, xacro)
@@ -97,5 +97,5 @@
     <parent link="base_link"/>
     <child link="lidar_rear"/>
-    <origin xyz="-0.288 -0.07 0.1" rpy="0 0 3.1415926535"/>
+    <origin xyz="-0.268 0.0 0.1" rpy="0 0 3.1415926535"/>
   </joint>
   <joint name="belt_launcher" type="continuous">

Commit message: fix tf

File: src/launch/krb2026b_launch/urdf/krb2026b.urdf.xacro (robot description, xacro)
@@ -99,4 +99,10 @@
     <origin xyz="-0.268 0.0 0.1" rpy="0 0 3.1415926535"/>
   </joint>
+  <link name="camera_link"/>
+  <joint name="base_link_to_camera_link" type="fixed">
+    <parent link="base_link"/>
+    <child link="camera_link"/>
+    <origin xyz="0.262 0 0.231" rpy="0 0 0"/>
+  </joint>
   <joint name="belt_launcher" type="continuous">
     <origin xyz="-0.15555731148 0.0 0.18967226953" rpy="0.0 -0.43633231299 0.0"/>

Commit message: 実機

File: src/launch/krb2026b_launch/urdf/krb2026b.urdf.xacro (robot description, xacro)
@@ -97,5 +97,5 @@
     <parent link="base_link"/>
     <child link="lidar_rear"/>
-    <origin xyz="-0.268 0.0 0.1" rpy="0 0 3.1415926535"/>
+    <origin xyz="-0.269 0.0 0.1" rpy="0 0 3.1415926535"/>
   </joint>
   <link name="camera_link"/>

Commit message: 実機

File: src/launch/krb2026b_launch/urdf/krb2026b.urdf.xacro (robot description, xacro)
@@ -184,3 +184,11 @@
     </visual>
   </link>
+  <link name="helper_link"/>
+  <joint name="helper" type="revolute">
+    <parent link="base_link"/>
+    <child link="helper_link"/>
+    <origin xyz="0.36669 0.0 0.4162" rpy="0 0 0"/>
+    <axis xyz="0 1 0"/>
+    <limit lower="-3.14159" upper="3.14159" effort="0" velocity="0"/>
+  </joint>
 </robot>
